File: attinyArcade/KiCAD/attinyArcade/attinyArcade.kicad_pcb (KiCad board)
At the start: 2 copper layers, 27.9 x 41.9 mm, 7 parts, among them SW1 SW_Push, SW2 SW_Push, U1 ATtiny85-20PU, U2 SSD1306_I2C_display

Commit message: arcade
Parts:
- added LS1: Speaker, My_Misc:Buzzer_TDK_PS1240P02BT_D12.2mm_H6.5mm_large, F.Cu at (177.8, 41.9)
- U1: value ATtiny85-20PU -> ATtiny85-20P; footprint My_Misc:DIP-8_W7.62mm_large -> My_Misc:DIP-8_W7.62mm_Socket_w_dip_packet_LongPads
- moved U1 0.47 mm to (148.0, 67.3)
Connections:
- U1 pad 1: Net-(U1-Pad1) -> unconnected-(U1-Pad1)
Other:
- net class Default removed
