File: attinyArcade/KiCAD/attinyArcade/attinyArcade.kicad_sch (KiCad schematic)
At the start: 8 parts

Commit message: kicad6
Parts:
- BT1: value (none) -> 3V; footprint (none) -> Battery:BatteryHolder_Keystone_103_1x20mm
- LS1: value (none) -> Speaker; footprint (none) -> My_Misc:Buzzer_TDK_PS1240P02BT_D12.2mm_H6.5mm_large
- R1, R2: value (none) -> 10k; footprint (none) -> My_Misc:R_Axial_DIN0207_L6.3mm_D2.5mm_P2.54mm_Vertical_large
- SW1, SW2: value (none) -> SW_Push; footprint (none) -> My_Misc:SW_PUSH_6mm_large
- U1: value (none) -> ATtiny85-20P; footprint (none) -> My_Misc:DIP-8_W7.62mm_Socket_w_dip_packet_LongPads
- U2: value (none) -> SSD1306_I2C_display; footprint (none) -> My_Parts:SSD1306_I2C_0.96_OLED_display_large
Changed lines of the file:
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@@
       (effects (font (size 1.27 1.27)) (justify left))
     )
-    (property "Value" "" (id 1) (at 47.4472 86.233 0)
+    (property "Value" "3V" (id 1) (at 47.4472 86.233 0)
       (effects (font (size 1.27 1.27)) (justify left))
     )
-    (property "Footprint" "" (id 2) (at 44.45 84.836 90)
+    (property "Footprint" "Battery:BatteryHolder_Keystone_103_1x20mm" (id 2) (at 44.45 84.836 90)
       (effects (font (size 1.27 1.27)) hide)
     )
@@
       (effects (font (size 1.27 1.27)) (justify left))
     )
-    (property "Value" "" (id 1) (at 159.258 101.473 0)
+    (property "Value" "Speaker" (id 1) (at 159.258 101.473 0)
       (effects (font (size 1.27 1.27)) (justify left))
     )
-    (property "Footprint" "" (id 2) (at 154.94 104.14 0)
+    (property "Footprint" "My_Misc:Buzzer_TDK_PS1240P02BT_D12.2mm_H6.5mm_large" (id 2) (at 154.94 104.14 0)
       (effects (font (size 1.27 1.27)) hide)
     )
@@
       (effects (font (size 1.27 1.27)) (justify left))
     )
-    (property "Value" "" (id 1) (at 116.7892 74.803 90)
+    (property "Value" "SW_Push" (id 1) (at 116.7892 74.803 90)
       (effects (font (size 1.27 1.27)) (justify left))
     )
-    (property "Footprint" "" (id 2) (at 118.11 73.66 0)
+    (property "Footprint" "My_Misc:SW_PUSH_6mm_large" (id 2) (at 118.11 73.66 0)
       (effects (font (size 1.27 1.27)) hide)
     )
@@
       (effects (font (size 1.27 1.27)) (justify left))
     )
-    (property "Value" "" (id 1) (at 132.0292 76.073 90)
+    (property "Value" "SW_Push" (id 1) (at 132.0292 76.073 90)
       (effects (font (size 1.27 1.27)) (justify left))
     )
-    (property "Footprint" "" (id 2) (at 133.35 74.93 0)
+    (property "Footprint" "My_Misc:SW_PUSH_6mm_large" (id 2) (at 133.35 74.93 0)
       (effects (font (size 1.27 1.27)) hide)
     )
@@
       (effects (font (size 1.27 1.27)) (justify left))
     )
-    (property "Value" "" (id 1) (at 114.808 88.773 0)
+    (property "Value" "10k" (id 1) (at 114.808 88.773 0)
       (effects (font (size 1.27 1.27)) (justify left))
     )
-    (property "Footprint" "" (id 2) (at 111.252 87.63 90)
+    (property "Footprint" "My_Misc:R_Axial_DIN0207_L6.3mm_D2.5mm_P2.54mm_Vertical_large" (id 2) (at 111.252 87.63 90)
       (effects (font (size 1.27 1.27)) hide)
     )
@@
       (effects (font (size 1.27 1.27)) (justify left))
     )
-    (property "Value" "" (id 1) (at 130.048 90.043 0)
+    (property "Value" "10k" (id 1) (at 130.048 90.043 0)
       (effects (font (size 1.27 1.27)) (justify left))
     )
-    (property "Footprint" "" (id 2) (at 126.492 88.9 90)
+    (property "Footprint" "My_Misc:R_Axial_DIN0207_L6.3mm_D2.5mm_P2.54mm_Vertical_large" (id 2) (at 126.492 88.9 90)
       (effects (font (size 1.27 1.27)) hide)
     )
@@
       (effects (font (size 1.27 1.27)) (justify left))
     )
-    (property "Value" "" (id 1) (at 170.8912 119.126 0)
+    (property "Value" "SSD1306_I2C_display" (id 1) (at 170.8912 119.126 0)
       (effects (font (size 1.27 1.27)) (justify left))
     )
-    (property "Footprint" "" (id 2) (at 154.305 111.76 0)
+    (property "Footprint" "My_Parts:SSD1306_I2C_0.96_OLED_display_large" (id 2) (at 154.305 111.76 0)
       (effects (font (size 1.27 1.27)) hide)
     )
@@
       (effects (font (size 1.27 1.27)) hide)
     )
-    (property "Value" "" (id 1) (at 82.677 113.6142 0))
+    (property "Value" "GND" (id 1) (at 82.677 113.6142 0))
     (property "Footprint" "" (id 2) (at 82.55 109.22 0)
       (effects (font (size 1.27 1.27)) hide)
@@
       (effects (font (size 1.27 1.27)) hide)
     )
-    (property "Value" "" (id 1) (at 137.287 132.6642 0))
+    (property "Value" "GND" (id 1) (at 137.287 132.6642 0))
     (property "Footprint" "" (id 2) (at 137.16 128.27 0)
       (effects (font (size 1.27 1.27)) hide)
@@
       (effects (font (size 1.27 1.27)) (justify right))
     )
-    (property "Value" "" (id 1) (at 69.088 85.5222 0)
+    (property "Value" "ATtiny85-20P" (id 1) (at 69.088 85.5222 0)
       (effects (font (size 1.27 1.27)) (justify right))
     )
-    (property "Footprint" "" (id 2) (at 82.55 83.82 0)
+    (property "Footprint" "My_Misc:DIP-8_W7.62mm_Socket_w_dip_packet_LongPads" (id 2) (at 82.55 83.82 0)
       (effects (font (size 1.27 1.27) italic) hide)
     )
