File: tinyTris/KiCAD/tinyTris/tinyTris.kicad_sch (KiCad schematic)
At the start: 15 parts

Commit message: kicad6
Parts:
- BT1: value (none) -> 3V; footprint (none) -> Battery:BatteryHolder_Keystone_103_1x20mm
- LS1: value (none) -> Piezo sound; footprint (none) -> My_Misc:Buzzer_TDK_PS1240P02BT_D12.2mm_H6.5mm_large
- R1, R4, R5: value (none) -> 10k; footprint (none) -> My_Misc:R_Axial_DIN0207_L6.3mm_D2.5mm_P10.16mm_Horizontal_larger_pads
- R2: value (none) -> 2k2; footprint (none) -> My_Misc:R_Axial_DIN0207_L6.3mm_D2.5mm_P10.16mm_Horizontal_larger_pads
- R3: value (none) -> 1k; footprint (none) -> My_Misc:R_Axial_DIN0207_L6.3mm_D2.5mm_P10.16mm_Horizontal_larger_pads
- SW1: value (none) -> Reset; footprint (none) -> My_Misc:SW_PUSH_6mm_large
- SW2: value (none) -> Rotate; footprint (none) -> My_Misc:SW_PUSH_6mm_large
- SW3: value (none) -> Left; footprint (none) -> My_Misc:SW_PUSH_6mm_large
- SW4: value (none) -> Right; footprint (none) -> My_Misc:SW_PUSH_6mm_large
- SW5: value (none) -> Drop; footprint (none) -> My_Misc:SW_PUSH_6mm_large
- U1: value (none) -> ATtiny85-20P; footprint (none) -> My_Misc:DIP-8_W7.62mm_Socket_w_dip_packet_LongPads
- U2: value (none) -> SSD1306_I2C_display; footprint (none) -> My_Parts:SSD1306_I2C_0.96_OLED_display_no_display_large
- U3: value (none) -> SSD1306_I2C_display; footprint (none) -> My_Parts:SSD1306_I2C_0.96_OLED_display_large
Changed lines of the file:
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@@
       (effects (font (size 1.27 1.27)) (justify left))
     )
-    (property "Value" "" (id 1) (at 276.098 101.473 0)
-      (effects (font (size 1.27 1.27)) (justify left))
-    )
-    (property "Footprint" "" (id 2) (at 271.78 104.14 0)
+    (property "Value" "Piezo sound" (id 1) (at 276.098 101.473 0)
+      (effects (font (size 1.27 1.27)) (justify left))
+    )
+    (property "Footprint" "My_Misc:Buzzer_TDK_PS1240P02BT_D12.2mm_H6.5mm_large" (id 2) (at 271.78 104.14 0)
       (effects (font (size 1.27 1.27)) hide)
     )
@@
       (effects (font (size 1.27 1.27)) (justify left))
     )
-    (property "Value" "" (id 1) (at 217.1192 72.263 90)
-      (effects (font (size 1.27 1.27)) (justify left))
-    )
-    (property "Footprint" "" (id 2) (at 218.44 71.12 0)
+    (property "Value" "Rotate" (id 1) (at 217.1192 72.263 90)
+      (effects (font (size 1.27 1.27)) (justify left))
+    )
+    (property "Footprint" "My_Misc:SW_PUSH_6mm_large" (id 2) (at 218.44 71.12 0)
       (effects (font (size 1.27 1.27)) hide)
     )
@@
       (effects (font (size 1.27 1.27)) (justify left))
     )
-    (property "Value" "" (id 1) (at 229.8192 72.263 90)
-      (effects (font (size 1.27 1.27)) (justify left))
-    )
-    (property "Footprint" "" (id 2) (at 231.14 71.12 0)
+    (property "Value" "Left" (id 1) (at 229.8192 72.263 90)
+      (effects (font (size 1.27 1.27)) (justify left))
+    )
+    (property "Footprint" "My_Misc:SW_PUSH_6mm_large" (id 2) (at 231.14 71.12 0)
       (effects (font (size 1.27 1.27)) hide)
     )
@@
       (effects (font (size 1.27 1.27)) (justify left))
     )
-    (property "Value" "" (id 1) (at 242.5192 72.263 90)
-      (effects (font (size 1.27 1.27)) (justify left))
-    )
-    (property "Footprint" "" (id 2) (at 243.84 71.12 0)
+    (property "Value" "Right" (id 1) (at 242.5192 72.263 90)
+      (effects (font (size 1.27 1.27)) (justify left))
+    )
+    (property "Footprint" "My_Misc:SW_PUSH_6mm_large" (id 2) (at 243.84 71.12 0)
       (effects (font (size 1.27 1.27)) hide)
     )
@@
       (effects (font (size 1.27 1.27)) (justify left))
     )
-    (property "Value" "" (id 1) (at 255.2192 72.263 90)
-      (effects (font (size 1.27 1.27)) (justify left))
-    )
-    (property "Footprint" "" (id 2) (at 256.54 71.12 0)
+    (property "Value" "Drop" (id 1) (at 255.2192 72.263 90)
+      (effects (font (size 1.27 1.27)) (justify left))
+    )
+    (property "Footprint" "My_Misc:SW_PUSH_6mm_large" (id 2) (at 256.54 71.12 0)
       (effects (font (size 1.27 1.27)) hide)
     )
@@
       (effects (font (size 1.27 1.27)) (justify left))
     )
-    (property "Value" "" (id 1) (at 227.838 58.293 0)
-      (effects (font (size 1.27 1.27)) (justify left))
-    )
-    (property "Footprint" "" (id 2) (at 224.282 57.15 90)
+    (property "Value" "2k2" (id 1) (at 227.838 58.293 0)
+      (effects (font (size 1.27 1.27)) (justify left))
+    )
+    (property "Footprint" "My_Misc:R_Axial_DIN0207_L6.3mm_D2.5mm_P10.16mm_Horizontal_larger_pads" (id 2) (at 224.282 57.15 90)
       (effects (font (size 1.27 1.27)) hide)
     )
@@
       (effects (font (size 1.27 1.27)) (justify left))
     )
-    (property "Value" "" (id 1) (at 240.538 58.293 0)
-      (effects (font (size 1.27 1.27)) (justify left))
-    )
-    (property "Footprint" "" (id 2) (at 236.982 57.15 90)
+    (property "Value" "1k" (id 1) (at 240.538 58.293 0)
+      (effects (font (size 1.27 1.27)) (justify left))
+    )
+    (property "Footprint" "My_Misc:R_Axial_DIN0207_L6.3mm_D2.5mm_P10.16mm_Horizontal_larger_pads" (id 2) (at 236.982 57.15 90)
       (effects (font (size 1.27 1.27)) hide)
     )
@@
       (effects (font (size 1.27 1.27)) (justify left))
     )
-    (property "Value" "" (id 1) (at 253.238 101.473 0)
-      (effects (font (size 1.27 1.27)) (justify left))
-    )
-    (property "Footprint" "" (id 2) (at 249.682 100.33 90)
+    (property "Value" "10k" (id 1) (at 253.238 101.473 0)
+      (effects (font (size 1.27 1.27)) (justify left))
+    )
+    (property "Footprint" "My_Misc:R_Axial_DIN0207_L6.3mm_D2.5mm_P10.16mm_Horizontal_larger_pads" (id 2) (at 249.682 100.33 90)
       (effects (font (size 1.27 1.27)) hide)
     )
@@
       (effects (font (size 1.27 1.27)) (justify left))
     )
-    (property "Value" "" (id 1) (at 70.3072 95.123 0)
-      (effects (font (size 1.27 1.27)) (justify left))
-    )
-    (property "Footprint" "" (id 2) (at 67.31 93.726 90)
+    (property "Value" "3V" (id 1) (at 70.3072 95.123 0)
+      (effects (font (size 1.27 1.27)) (justify left))
+    )
+    (property "Footprint" "Battery:BatteryHolder_Keystone_103_1x20mm" (id 2) (at 67.31 93.726 90)
       (effects (font (size 1.27 1.27)) hide)
     )
@@
       (effects (font (size 1.27 1.27)) (justify left))
     )
-    (property "Value" "" (id 1) (at 204.4192 115.443 90)
-      (effects (font (size 1.27 1.27)) (justify left))
-    )
-    (property "Footprint" "" (id 2) (at 205.74 114.3 0)
+    (property "Value" "Reset" (id 1) (at 204.4192 115.443 90)
+      (effects (font (size 1.27 1.27)) (justify left))
+    )
+    (property "Footprint" "My_Misc:SW_PUSH_6mm_large" (id 2) (at 205.74 114.3 0)
       (effects (font (size 1.27 1.27)) hide)
     )
@@
       (effects (font (size 1.27 1.27)) hide)
     )
-    (property "Value" "" (id 1) (at 200.787 128.8542 0))
+    (property "Value" "GND" (id 1) (at 200.787 128.8542 0))
     (property "Footprint" "" (id 2) (at 200.66 124.46 0)
       (effects (font (size 1.27 1.27)) hide)
@@
       (effects (font (size 1.27 1.27)) hide)
     )
-    (property "Value" "" (id 1) (at 109.347 128.8542 0))
+    (property "Value" "GND" (id 1) (at 109.347 128.8542 0))
     (property "Footprint" "" (id 2) (at 109.22 124.46 0)
       (effects (font (size 1.27 1.27)) hide)
@@
       (effects (font (size 1.27 1.27)) hide)
     )
-    (property "Value" "" (id 1) (at 251.587 128.8542 0))
+    (property "Value" "GND" (id 1) (at 251.587 128.8542 0))
     (property "Footprint" "" (id 2) (at 251.46 124.46 0)
       (effects (font (size 1.27 1.27)) hide)
@@
       (effects (font (size 1.27 1.27)) (justify left))
     )
-    (property "Value" "" (id 1) (at 240.538 101.473 0)
-      (effects (font (size 1.27 1.27)) (justify left))
-    )
-    (property "Footprint" "" (id 2) (at 236.982 100.33 90)
+    (property "Value" "10k" (id 1) (at 240.538 101.473 0)
+      (effects (font (size 1.27 1.27)) (justify left))
+    )
+    (property "Footprint" "My_Misc:R_Axial_DIN0207_L6.3mm_D2.5mm_P10.16mm_Horizontal_larger_pads" (id 2) (at 236.982 100.33 90)
       (effects (font (size 1.27 1.27)) hide)
     )
@@
       (effects (font (size 1.27 1.27)) hide)
     )
-    (property "Value" "" (id 1) (at 238.887 128.8542 0))
+    (property "Value" "GND" (id 1) (at 238.887 128.8542 0))
     (property "Footprint" "" (id 2) (at 238.76 124.46 0)
       (effects (font (size 1.27 1.27)) hide)
@@
       (effects (font (size 1.27 1.27)) hide)
     )
-    (property "Value" "" (id 1) (at 261.747 128.8542 0))
+    (property "Value" "GND" (id 1) (at 261.747 128.8542 0))
     (property "Footprint" "" (id 2) (at 261.62 124.46 0)
       (effects (font (size 1.27 1.27)) hide)
@@
     (in_bom yes) (on_board yes)
     (property "Reference" "U2" (id 0) (at 165.5318 106.299 0))
-    (property "Value" "" (id 1) (at 165.5318 108.6104 0))
-    (property "Footprint" "" (id 2) (at 160.655 121.92 0)
+    (property "Value" "SSD1306_I2C_display" (id 1) (at 165.5318 108.6104 0))
+    (property "Footprint" "My_Parts:SSD1306_I2C_0.96_OLED_display_no_display_large" (id 2) (at 160.655 121.92 0)
       (effects (font (size 1.27 1.27)) hide)
     )
@@
       (effects (font (size 1.27 1.27)) hide)
     )
-    (property "Value" "" (id 1) (at 133.477 130.1242 0))
+    (property "Value" "GND" (id 1) (at 133.477 130.1242 0))
     (property "Footprint" "" (id 2) (at 133.35 125.73 0)
       (effects (font (size 1.27 1.27)) hide)
@@
       (effects (font (size 1.27 1.27)) (justify left))
     )
-    (property "Value" "" (id 1) (at 202.438 73.533 0)
-      (effects (font (size 1.27 1.27)) (justify left))
-    )
-    (property "Footprint" "" (id 2) (at 198.882 72.39 90)
+    (property "Value" "10k" (id 1) (at 202.438 73.533 0)
+      (effects (font (size 1.27 1.27)) (justify left))
+    )
+    (property "Footprint" "My_Misc:R_Axial_DIN0207_L6.3mm_D2.5mm_P10.16mm_Horizontal_larger_pads" (id 2) (at 198.882 72.39 90)
       (effects (font (size 1.27 1.27)) hide)
     )
@@
       (effects (font (size 1.27 1.27)) (justify left))
     )
-    (property "Value" "" (id 1) (at 177.2412 131.826 0)
-      (effects (font (size 1.27 1.27)) (justify left))
-    )
-    (property "Footprint" "" (id 2) (at 160.655 124.46 0)
+    (property "Value" "SSD1306_I2C_display" (id 1) (at 177.2412 131.826 0)
+      (effects (font (size 1.27 1.27)) (justify left))
+    )
+    (property "Footprint" "My_Parts:SSD1306_I2C_0.96_OLED_display_large" (id 2) (at 160.655 124.46 0)
       (effects (font (size 1.27 1.27)) hide)
     )
@@
       (effects (font (size 1.27 1.27)) (justify right))
     )
-    (property "Value" "" (id 1) (at 95.758 95.6822 0)
+    (property "Value" "ATtiny85-20P" (id 1) (at 95.758 95.6822 0)
       (effects (font (size 1.27 1.27)) (justify right))
     )
-    (property "Footprint" "" (id 2) (at 109.22 93.98 0)
+    (property "Footprint" "My_Misc:DIP-8_W7.62mm_Socket_w_dip_packet_LongPads" (id 2) (at 109.22 93.98 0)
       (effects (font (size 1.27 1.27) italic) hide)
     )

Commit message: new schematics
Connections:
- net GND: now also U3.1 (GND); no longer U3.4 (SDA)
- net at BT1.1 (+), R1.1, R2.1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: now also U3.2 (VCC); no longer U3.3 (SCL)
- net at U1.3 (XTAL2/PB4), U2.3 (SCL): now also U3.3 (SCL); no longer U3.2 (VCC)
- net at U1.2 (XTAL1/PB3), U2.4 (SDA): now also U3.4 (SDA); no longer U3.1 (GND)
Other:
- moved on the sheet: BT1, LS1, R1, R2, R3, R4, R5, SW1, SW2, SW3, SW4, SW5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
